File: CX_buttonlight_v2.kicad_pcb (KiCad board)
At the start: 2 copper layers, 20 x 15 mm, 14 parts, among them U1 LM317LIPK

Commit message: Fuse added, minor fix in link given in README.md fixed
Parts:
- added F1: Fuse, Fuse:Fuse_0805_2012Metric_Pad1.15x1.40mm_HandSolder, B.Cu at (112.5, 60.9)
- R2: value 560R -> 536R
Connections:
- Supply1 pad 1: Net-(D4-~_2) -> Net-(F1-Pad1)
- TP1 pad 1: Net-(D4-~_2) -> Net-(F1-Pad1)
- TP2 pad 1: Net-(D4-~_2) -> Net-(F1-Pad1)
Routing:
- net Net-(D4-~_2): track 14.0 -> 2.82 mm
- net Net-(F1-Pad1): track 0.00 -> 10.3 mm
Other:
- board text added: "PowerStation 2025 v1.3"
- board text removed: "PowerStation 2025 v1.2"
